Commit message: new change

File: src/my_robot/urdf/turtlebot3_with_sensors.urdf (robot description, URDF)
Before this commit: robot turtlebot3_waffle, 16 links, 15 joints
Links:
- removed link ${namespace}base_footprint
- removed link ${namespace}base_link
- removed link ${namespace}base_scan
- removed link ${namespace}camera_depth_frame
- removed link ${namespace}camera_depth_optical_frame
- removed link ${namespace}camera_link
- removed link ${namespace}camera_rgb_frame
- removed link ${namespace}camera_rgb_optical_frame
- removed link ${namespace}caster_back_left_link
- removed link ${namespace}caster_back_right_link
- removed link ${namespace}imu_link
- removed link ${namespace}wheel_left_link
- removed link ${namespace}wheel_right_link
- removed link camera_back_link
- removed link camera_front_link
- removed link lidar3d_link
- added link base_footprint
- added link base_link, mass 1.0; collision box size=0.266 0.266 0.094; visual mesh filename=package://turtlebot3_description/meshes/bases/waffle_base.s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 scale=0.001 0.001 0.001
- added link base_scan, mass 0.114; collision cylinder length=0.0315 radius=0.055; visual cylinder length=0.0315 radius=0.055
- added link camera_left_link, mass 0.01
- added link camera_right_link, mass 0.01
- added link caster_back_left_link, mass 0.01
- added link caster_back_right_link, mass 0.01
- added link velodyne_link, mass 0.83; collision cylinder length=0.07 radius=0.05; visual cylinder length=0.07 radius=0.05
- added link wheel_left_link, mass 0.1; collision cylinder length=0.018 radius=0.033; visual mesh filename=package://turtlebot3_description/meshes/wheels/left_tire.stl scale=0.001 0.001 0.001
- added link wheel_right_link, mass 0.1; collision cylinder length=0.018 radius=0.033; visual mesh filename=package://turtlebot3_description/meshes/wheels/right_tire.s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 scale=0.001 0.001 0.001
Joints:
- removed joint ${namespace}base_joint
- removed joint ${namespace}camera_depth_joint
- removed joint ${namespace}camera_depth_optical_joint
- removed joint ${namespace}camera_joint
- removed joint ${namespace}camera_rgb_joint
- removed joint ${namespace}camera_rgb_optical_joint
- removed joint ${namespace}caster_back_left_joint
- removed joint ${namespace}caster_back_right_joint
- removed joint ${namespace}imu_joint
- removed joint ${namespace}scan_joint
- removed joint ${namespace}wheel_left_joint
- removed joint ${namespace}wheel_right_joint
- removed joint camera_back_joint
- removed joint camera_front_joint
- removed joint lidar3d_joint
- added joint base_joint: type fixed, parent base_footprint, child base_link, origin xyz=0 0 0.010 rpy=0 0 0
- added joint camera_left_joint: type fixed, parent base_link, child camera_left_link, origin xyz=0.12 0.05 0.25 rpy=0 0 0
- added joint camera_right_joint: type fixed, parent base_link, child camera_right_link, origin xyz=0.12 -0.05 0.25 rpy=0 0 0
- added joint caster_back_left_joint: type fixed, parent base_link, child caster_back_left_link, origin xyz=-0.177 0.064 -0.004 rpy=-1.57 0 0
- added joint caster_back_right_joint: type fixed, parent base_link, child caster_back_right_link, origin xyz=-0.177 -0.064 -0.004 rpy=-1.57 0 0
- added joint scan_joint: type fixed, parent base_link, child base_scan, origin xyz=-0.064 0 0.122 rpy=0 0 0
- added joint velodyne_joint: type fixed, parent base_link, child velodyne_link, origin xyz=0 0 0.35 rpy=0 0 0
- added joint wheel_left_joint: type continuous, parent base_link, child wheel_left_link, origin xyz=0.0 0.144 0.023 rpy=-1.57 0 0, axis 0 0 1
- added joint wheel_right_joint: type continuous, parent base_link, child wheel_right_link, origin xyz=0.0 -0.144 0.023 rpy=-1.57 0 0, axis 0 0 1

Commit message: Add SLAM + Nav2 integration setup with goal_bridge and launch files

File: src/my_robot/urdf/turtlebot3_with_sensors.urdf (robot description, URDF)
Before this commit: robot turtlebot3_waffle, 10 links, 9 joints
Joints:
- joint velodyne_joint: origin xyz=0 0 0.35 rpy=0 0 0 -> xyz=0 0 0.18 rpy=0 0 0
